File: fuenteSimetrica/fuenteSimetrica2.brd (EAGLE design)
At the start: 100 x 80 mm, 26 parts, among them IC1 317T, IC2 337T

Commit message: Fuente Simétrica
Parts:
- moved R6 54.6 mm to (22.9, 43.2), turned to 270 degrees
- moved R8 38.2 mm to (69.8, 45.7), turned to 180 degrees
- moved IC2 23.4 mm to (52.1, 69.8)
- moved C2 17.0 mm to (16.5, 8.89)
- moved C8 16.7 mm to (64.8, 36.8), turned to 180 degrees
- moved C6 15.3 mm to (5.08, 10.2), turned to 270 degrees
- moved D1 14.2 mm to (33.0, 61.0)
- moved D2 14.2 mm to (17.8, 61.0)
- moved D3 14.2 mm to (33.0, 54.6)
- moved D4 14.2 mm to (17.8, 54.6)
- moved C5 11.7 mm to (5.08, 64.8), turned to 270 degrees
- moved R7 11.5 mm to (27.9, 68.6), turned to 0 degrees
- moved C3 11.4 mm to (45.7, 36.8), turned to 180 degrees
- moved C7 11.4 mm to (55.9, 36.8), turned to 180 degrees
- moved IC1 11.4 mm to (64.8, 69.8)
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Connections:
- removed net N$13: C2.-, C6.2, D3.A, D4.A, IC2.2, R8.1
- net GND: now also C2.-, C6.2, D3.A, D4.A, IC2.2, R8.1; no longer SALIDA.2
Routing:
- net N$5: track 117.6 -> 0.00 mm
- net N$13: track 95.2 -> 0.00 mm
- net N$2: track 82.6 -> 0.00 mm
- net N$9: track 50.7 -> 0.00 mm
- net N$10: track 45.6 -> 0.00 mm
- net N$1: track 45.1 -> 0.00 mm
- net N$12: track 37.4 -> 0.00 mm
- net N$3: track 28.8 -> 0.00 mm
- net N$7: track 12.3 -> 0.00 mm
- net N$11: track 12.3 -> 0.00 mm
- net N$4: track 9.72 -> 0.00 mm
- net N$8: track 5.08 -> 0.00 mm
